File: bolt-esc.brd (EAGLE design)
At the start: 53.7 x 52.2 mm, 0 parts

Commit message: More board work
Other:
- board size 53.7 x 52.2 mm -> 53.7 x 63.7 mm
Changed lines of the file:
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@@
 <wire x1="72.27" y1="65.9" x2="72.27" y2="44.7" width="0.1524" layer="20"/>
 <wire x1="46.7" y1="80.6" x2="29.9" y2="88.8" width="0.1524" layer="20"/>
+<wire x1="51.8" y1="92.1" x2="35" y2="100.3" width="0.1524" layer="20"/>
 </plain>
 <attributes>
